File: Hardware/Relays.sch (KiCad schematic (older format))
At the start: 0 parts

Commit message: [Hardware] Added relays schematic sheet.
Parts:
- added D1, D2, D3, D4, D5, D6, D7, D8: BAT54C, Package_TO_SOT_SMD:SOT-23, symbol Diode:BAT54C
- added J1, J10, J11, J12, J13, J14, J15, J16, J2, J3, J4, J5, J6, J7, J8, J9: 282834-3, TerminalBlock_TE-Connectivity:TerminalBlock_TE_282834-3_1x03_P2.54mm_Horizontal, symbol Connector:Screw_Terminal_01x03
- added K1, K10, K11, K12, K13, K14, K15, K16, K2, K3, K4, K5, K6, K7, K8, K9: HRS1H-S_DC5V, HRS1H-S:HRS1H-S, symbol HRS1H-S:HRS1H-S_DC5V
- added Q1, Q10, Q11, Q12, Q13, Q14, Q15, Q16, Q2, Q3, Q4, Q5, Q6, Q7, Q8, Q9: BC848, Package_TO_SOT_SMD:SOT-23, symbol Transistor_BJT:BC848
- added R10, R11, R12, R13, R14, R15, R16, R17, R18, R3, R4, R5, R6, R7, R8, R9: 1K, Resistor_SMD:R_0603_1608Metric_Pad0.98x0.95mm_HandSolder, symbol Device:R
Connections:
- new net: J1.2 (Pin_2), K1.1
- new net: D1.2, K1.2, Q1.3 (C)
- new net: J1.1 (Pin_1), K1.3
- new net: J1.3 (Pin_3), K1.6
- new net: Q1.1 (B), R3.1
- new net: D1.1, K2.5, Q2.3 (C)
- new net: J2.2 (Pin_2), K2.1
- new net: J2.1 (Pin_1), K2.3
- new net: J2.3 (Pin_3), K2.6
- new net: Q2.1 (B), R4.1
- new net: J3.2 (Pin_2), K3.1
- new net: D2.2, K3.2, Q3.3 (C)
- new net: J3.1 (Pin_1), K3.3
- new net: J3.3 (Pin_3), K3.6
- new net: Q3.1 (B), R5.1
- new net: D2.1, K4.5, Q4.3 (C)
- new net: J4.2 (Pin_2), K4.1
- new net: J4.1 (Pin_1), K4.3
- new net: J4.3 (Pin_3), K4.6
- new net: Q4.1 (B), R6.1
- new net: J5.2 (Pin_2), K5.1
- new net: D3.2, K5.2, Q5.3 (C)
- new net: J5.1 (Pin_1), K5.3
- new net: J5.3 (Pin_3), K5.6
- new net: Q5.1 (B), R7.1
- new net: D3.1, K6.5, Q6.3 (C)
- new net: J6.2 (Pin_2), K6.1
- new net: J6.1 (Pin_1), K6.3
- new net: J6.3 (Pin_3), K6.6
- new net: Q6.1 (B), R8.1
- new net: J7.2 (Pin_2), K7.1
- new net: D4.2, K7.2, Q7.3 (C)
- new net: J7.1 (Pin_1), K7.3
- new net: J7.3 (Pin_3), K7.6
- new net: Q7.1 (B), R9.1
- new net: D4.1, K8.5, Q8.3 (C)
- new net: J8.2 (Pin_2), K8.1
- new net: J8.1 (Pin_1), K8.3
- new net: J8.3 (Pin_3), K8.6
- new net: Q8.1 (B), R10.1
- new net: J9.2 (Pin_2), K9.1
- new net: D5.2, K9.2, Q9.3 (C)
- new net: J9.1 (Pin_1), K9.3
- new net: J9.3 (Pin_3), K9.6
- new net: Q9.1 (B), R11.1
- new net: D5.1, K10.5, Q10.3 (C)
- new net: J10.2 (Pin_2), K10.1
- new net: J10.1 (Pin_1), K10.3
- new net: J10.3 (Pin_3), K10.6
- new net: Q10.1 (B), R12.1
- new net: J11.2 (Pin_2), K11.1
- new net: D6.2, K11.2, Q11.3 (C)
- new net: J11.1 (Pin_1), K11.3
- new net: J11.3 (Pin_3), K11.6
- new net: Q11.1 (B), R13.1
- new net: D6.1, K12.5, Q12.3 (C)
- new net: J12.2 (Pin_2), K12.1
- new net: J12.1 (Pin_1), K12.3
- new net: J12.3 (Pin_3), K12.6
- new net: Q12.1 (B), R14.1
- new net: J13.2 (Pin_2), K13.1
- new net: D7.2, K13.2, Q13.3 (C)
- new net: J13.1 (Pin_1), K13.3
- new net: J13.3 (Pin_3), K13.6
- new net: Q13.1 (B), R15.1
- new net: D7.1, K14.5, Q14.3 (C)
- new net: J14.2 (Pin_2), K14.1
- new net: J14.1 (Pin_1), K14.3
- new net: J14.3 (Pin_3), K14.6
- new net: Q14.1 (B), R16.1
- new net: J15.2 (Pin_2), K15.1
- new net: D8.2, K15.2, Q15.3 (C)
- new net: J15.1 (Pin_1), K15.3
- new net: J15.3 (Pin_3), K15.6
- new net: Q15.1 (B), R17.1
- new net: D8.1, K16.5, Q16.3 (C)
- new net: J16.2 (Pin_2), K16.1
- new net: J16.1 (Pin_1), K16.3
- new net: J16.3 (Pin_3), K16.6
- new net: Q16.1 (B), R18.1
- new net +5V: D1.3, D2.3, D3.3, D4.3, D5.3, D6.3, D7.3, D8.3, K1.5, K10.2, K11.5, K12.2, K13.5, K14.2, K15.5, K16.2, K2.2, K3.5, K4.2, K5.5, K6.2, K7.5, K8.2, K9.5
- new net GND: Q1.2 (E), Q10.2 (E), Q11.2 (E), Q12.2 (E), Q13.2 (E), Q14.2 (E), Q15.2 (E), Q16.2 (E), Q2.2 (E), Q3.2 (E), Q4.2 (E), Q5.2 (E), Q6.2 (E), Q7.2 (E), Q8.2 (E), Q9.2 (E)
- new net RELAY_1: R3.2
- new net RELAY_10: R12.2
- new net RELAY_11: R13.2
- new net RELAY_12: R14.2
- new net RELAY_13: R15.2
- new net RELAY_14: R16.2
- new net RELAY_15: R17.2
- new net RELAY_16: R18.2
- new net RELAY_2: R4.2
- new net RELAY_3: R5.2
- new net RELAY_4: R6.2
- new net RELAY_5: R7.2
- new net RELAY_6: R8.2
- new net RELAY_7: R9.2
- new net RELAY_8: R10.2
- new net RELAY_9: R11.2
- no-connect marks 0 -> 16
Other:
- note added: "BAT54C diodes are obsolete and can be replaced by BAT754C,\nbut they are currently cheaper."

Commit message: [Hardware] Added terminal 3D models.
Parts:
- J1, J10, J11, J12, J13, J14, J15, J16, J2, J3, J4, J5, J6, J7, J8, J9: footprint TerminalBlock_TE-Connectivity:TerminalBlock_TE_282834-3_1x03_P2.54mm_Horizontal -> 282834-3:TerminalBlock_TE_282834-3_1x03_P2.54mm_Horizontal
Changed lines of the file:
@@
 F 0 "J1" V 1564 1112 50  0000 R CNN
 F 1 "282834-3" V 1473 1112 50  0000 R CNN
-F 2 "TerminalBlock_TE-Connectivity:TerminalBlock_TE_282834-3_1x03_P2.54mm_Horizontal" H 1600 1300 50  0001 C CNN
+F 2 "282834-3:TerminalBlock_TE_282834-3_1x03_P2.54mm_Horizontal" H 1600 1300 50  0001 C CNN
 F 3 "~" H 1600 1300 50  0001 C CNN
 F 4 "TE" H 1600 1300 50  0001 C CNN "Manufacturer"
@@
 F 0 "J2" V 3664 1112 50  0000 R CNN
 F 1 "282834-3" V 3573 1112 50  0000 R CNN
-F 2 "TerminalBlock_TE-Connectivity:TerminalBlock_TE_282834-3_1x03_P2.54mm_Horizontal" H 3700 1300 50  0001 C CNN
+F 2 "282834-3:TerminalBlock_TE_282834-3_1x03_P2.54mm_Horizontal" H 3700 1300 50  0001 C CNN
 F 3 "~" H 3700 1300 50  0001 C CNN
 F 4 "TE" H 3700 1300 50  0001 C CNN "Manufacturer"
@@
 F 0 "J3" V 5414 1112 50  0000 R CNN
 F 1 "282834-3" V 5323 1112 50  0000 R CNN
-F 2 "TerminalBlock_TE-Connectivity:TerminalBlock_TE_282834-3_1x03_P2.54mm_Horizontal" H 5450 1300 50  0001 C CNN
+F 2 "282834-3:TerminalBlock_TE_282834-3_1x03_P2.54mm_Horizontal" H 5450 1300 50  0001 C CNN
 F 3 "~" H 5450 1300 50  0001 C CNN
 F 4 "TE" H 5450 1300 50  0001 C CNN "Manufacturer"
@@
 F 0 "J4" V 7514 1112 50  0000 R CNN
 F 1 "282834-3" V 7423 1112 50  0000 R CNN
-F 2 "TerminalBlock_TE-Connectivity:TerminalBlock_TE_282834-3_1x03_P2.54mm_Horizontal" H 7550 1300 50  0001 C CNN
+F 2 "282834-3:TerminalBlock_TE_282834-3_1x03_P2.54mm_Horizontal" H 7550 1300 50  0001 C CNN
 F 3 "~" H 7550 1300 50  0001 C CNN
 F 4 "TE" H 7550 1300 50  0001 C CNN "Manufacturer"
@@
 F 0 "J5" V 9264 1112 50  0000 R CNN
 F 1 "282834-3" V 9173 1112 50  0000 R CNN
-F 2 "TerminalBlock_TE-Connectivity:TerminalBlock_TE_282834-3_1x03_P2.54mm_Horizontal" H 9300 1300 50  0001 C CNN
+F 2 "282834-3:TerminalBlock_TE_282834-3_1x03_P2.54mm_Horizontal" H 9300 1300 50  0001 C CNN
 F 3 "~" H 9300 1300 50  0001 C CNN
 F 4 "TE" H 9300 1300 50  0001 C CNN "Manufacturer"
@@
 F 0 "J6" V 11364 1112 50  0000 R CNN
 F 1 "282834-3" V 11273 1112 50  0000 R CNN
-F 2 "TerminalBlock_TE-Connectivity:TerminalBlock_TE_282834-3_1x03_P2.54mm_Horizontal" H 11400 1300 50  0001 C CNN
+F 2 "282834-3:TerminalBlock_TE_282834-3_1x03_P2.54mm_Horizontal" H 11400 1300 50  0001 C CNN
 F 3 "~" H 11400 1300 50  0001 C CNN
 F 4 "TE" H 11400 1300 50  0001 C CNN "Manufacturer"
@@
 F 0 "J7" V 13014 1112 50  0000 R CNN
 F 1 "282834-3" V 12923 1112 50  0000 R CNN
-F 2 "TerminalBlock_TE-Connectivity:TerminalBlock_TE_282834-3_1x03_P2.54mm_Horizontal" H 13050 1300 50  0001 C CNN
+F 2 "282834-3:TerminalBlock_TE_282834-3_1x03_P2.54mm_Horizontal" H 13050 1300 50  0001 C CNN
 F 3 "~" H 13050 1300 50  0001 C CNN
 F 4 "TE" H 13050 1300 50  0001 C CNN "Manufacturer"
@@
 F 0 "J8" V 15114 1112 50  0000 R CNN
 F 1 "282834-3" V 15023 1112 50  0000 R CNN
-F 2 "TerminalBlock_TE-Connectivity:TerminalBlock_TE_282834-3_1x03_P2.54mm_Horizontal" H 15150 1300 50  0001 C CNN
+F 2 "282834-3:TerminalBlock_TE_282834-3_1x03_P2.54mm_Horizontal" H 15150 1300 50  0001 C CNN
 F 3 "~" H 15150 1300 50  0001 C CNN
 F 4 "TE" H 15150 1300 50  0001 C CNN "Manufacturer"
@@
 F 0 "J9" V 1564 5462 50  0000 R CNN
 F 1 "282834-3" V 1473 5462 50  0000 R CNN
-F 2 "TerminalBlock_TE-Connectivity:TerminalBlock_TE_282834-3_1x03_P2.54mm_Horizontal" H 1600 5650 50  0001 C CNN
+F 2 "282834-3:TerminalBlock_TE_282834-3_1x03_P2.54mm_Horizontal" H 1600 5650 50  0001 C CNN
 F 3 "~" H 1600 5650 50  0001 C CNN
 F 4 "TE" H 1600 5650 50  0001 C CNN "Manufacturer"
@@
 F 0 "J10" V 3664 5462 50  0000 R CNN
 F 1 "282834-3" V 3573 5462 50  0000 R CNN
-F 2 "TerminalBlock_TE-Connectivity:TerminalBlock_TE_282834-3_1x03_P2.54mm_Horizontal" H 3700 5650 50  0001 C CNN
+F 2 "282834-3:TerminalBlock_TE_282834-3_1x03_P2.54mm_Horizontal" H 3700 5650 50  0001 C CNN
 F 3 "~" H 3700 5650 50  0001 C CNN
 F 4 "TE" H 3700 5650 50  0001 C CNN "Manufacturer"
@@
 F 0 "J11" V 5414 5462 50  0000 R CNN
 F 1 "282834-3" V 5323 5462 50  0000 R CNN
-F 2 "TerminalBlock_TE-Connectivity:TerminalBlock_TE_282834-3_1x03_P2.54mm_Horizontal" H 5450 5650 50  0001 C CNN
+F 2 "282834-3:TerminalBlock_TE_282834-3_1x03_P2.54mm_Horizontal" H 5450 5650 50  0001 C CNN
 F 3 "~" H 5450 5650 50  0001 C CNN
 F 4 "TE" H 5450 5650 50  0001 C CNN "Manufacturer"
@@
 F 0 "J12" V 7514 5462 50  0000 R CNN
 F 1 "282834-3" V 7423 5462 50  0000 R CNN
-F 2 "TerminalBlock_TE-Connectivity:TerminalBlock_TE_282834-3_1x03_P2.54mm_Horizontal" H 7550 5650 50  0001 C CNN
+F 2 "282834-3:TerminalBlock_TE_282834-3_1x03_P2.54mm_Horizontal" H 7550 5650 50  0001 C CNN
 F 3 "~" H 7550 5650 50  0001 C CNN
 F 4 "TE" H 7550 5650 50  0001 C CNN "Manufacturer"
@@
 F 0 "J13" V 9264 5462 50  0000 R CNN
 F 1 "282834-3" V 9173 5462 50  0000 R CNN
-F 2 "TerminalBlock_TE-Connectivity:TerminalBlock_TE_282834-3_1x03_P2.54mm_Horizontal" H 9300 5650 50  0001 C CNN
+F 2 "282834-3:TerminalBlock_TE_282834-3_1x03_P2.54mm_Horizontal" H 9300 5650 50  0001 C CNN
 F 3 "~" H 9300 5650 50  0001 C CNN
 F 4 "TE" H 9300 5650 50  0001 C CNN "Manufacturer"
@@
 F 0 "J14" V 11364 5462 50  0000 R CNN
 F 1 "282834-3" V 11273 5462 50  0000 R CNN
-F 2 "TerminalBlock_TE-Connectivity:TerminalBlock_TE_282834-3_1x03_P2.54mm_Horizontal" H 11400 5650 50  0001 C CNN
+F 2 "282834-3:TerminalBlock_TE_282834-3_1x03_P2.54mm_Horizontal" H 11400 5650 50  0001 C CNN
 F 3 "~" H 11400 5650 50  0001 C CNN
 F 4 "TE" H 11400 5650 50  0001 C CNN "Manufacturer"
@@
 F 0 "J15" V 13014 5462 50  0000 R CNN
 F 1 "282834-3" V 12923 5462 50  0000 R CNN
-F 2 "TerminalBlock_TE-Connectivity:TerminalBlock_TE_282834-3_1x03_P2.54mm_Horizontal" H 13050 5650 50  0001 C CNN
+F 2 "282834-3:TerminalBlock_TE_282834-3_1x03_P2.54mm_Horizontal" H 13050 5650 50  0001 C CNN
 F 3 "~" H 13050 5650 50  0001 C CNN
 F 4 "TE" H 13050 5650 50  0001 C CNN "Manufacturer"
@@
 F 0 "J16" V 15114 5462 50  0000 R CNN
 F 1 "282834-3" V 15023 5462 50  0000 R CNN
-F 2 "TerminalBlock_TE-Connectivity:TerminalBlock_TE_282834-3_1x03_P2.54mm_Horizontal" H 15150 5650 50  0001 C CNN
+F 2 "282834-3:TerminalBlock_TE_282834-3_1x03_P2.54mm_Horizontal" H 15150 5650 50  0001 C CNN
 F 3 "~" H 15150 5650 50  0001 C CNN
 F 4 "TE" H 15150 5650 50  0001 C CNN "Manufacturer"

Commit message: [Hardware] Renamed components in a more coherent way.
Parts:
- renumbered R3 to R1, R12 to R10, R13 to R11, R14 to R12, R15 to R13, R16 to R14, R17 to R15, R18 to R16, R4 to R2, R5 to R3, R6 to R4, R7 to R5, R8 to R6, R9 to R7, R10 to R8, R11 to R9
