File: Hardware/USB_Relays.kicad_pcb (KiCad board)
At the start: 2 copper layers, 94 x 130.8 mm, 94 parts, among them J1 282834-3, J10 282834-3, J11 282834-3, J12 282834-3, J13 282834-3, J14 282834-3, J15 282834-3, J16 282834-3, J17 DNP, J18 2411_06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

Commit message: [Hardware] Inverted relays 'NC' and 'NO' markings on PC silkscreen to match real relay internal connections.
Other:
- board text added: "~MCLR~"
